Commit message: Project completed: version 1.0

File: mobilebot_description/urdf/kinect.xacro (robot description, xacro)
@@ -13,11 +13,11 @@
     xmlns:physics="http://playerstage.sourceforge.net/gazebo/xmlschema/#physics"
     xmlns:xacro="https://www.ros.org/wiki/xacro">
-  <!-- math constants -->
+ <!-- math constants -->
   <xacro:property name="M_PI" value="3.1415926535897931" />
-  <xacro:macro name="kinect" params="xyz parent_frame" >
+  <xacro:macro name="kinect" params="xyz rpy parent_frame" >
   <joint name="base_camera_joint" type="fixed">
-    <axis xyz="0 1 0" />
-    <origin xyz="${xyz}" rpy="0.0 0.0 0.0" />
+    <origin xyz="${xyz}" rpy="${rpy}" />
     <parent link="${parent_frame}" />
+    <origin xyz="0 0 0" rpy="0 0 0" />
     <child link="camera_link" />
   </joint>
@@ -31,5 +31,5 @@
     </inertial>
     <visual>
-      <origin xyz=" 0 0 0 " rpy="0 0 1.570796327" />
+      <origin xyz=" 0 0 0 " rpy="0 0 0" />
       <geometry>
         <mesh filename="package://mobilebot_description/meshes/kinect.dae"/>
@@ -39,5 +39,5 @@
       <origin xyz="0.0 0.0 0.0" rpy="0 0 0" />
       <geometry>
-        <box size="0.0730 0.2760 0.0720"/>
+        <box size="0.0730 .2760 0.0720"/>
       </geometry>
     </collision>
@@ -58,5 +58,5 @@
   </link>
   <joint name="camera_depth_optical_joint" type="fixed">
-    <origin xyz="0 0 0" rpy="0 0 0" />
+    <origin xyz="0 0 0" rpy="${-M_PI/2} 0 ${-M_PI/2}" />
     <parent link="camera_depth_frame" />
     <child link="camera_depth_optical_frame" />
@@ -73,5 +73,5 @@
   <joint name="camera_rgb_joint" type="fixed">
     <origin xyz="0 -0.012 0" rpy="0 0 0" />
-    <parent link="camera_depth_frame" />
+    <parent link="camera_link" />
     <child link="camera_rgb_frame" />
   </joint>
@@ -86,5 +86,5 @@
   </link>
   <joint name="camera_rgb_optical_joint" type="fixed">
-    <origin xyz="0 0 0" rpy="0 0 0" />
+    <origin xyz="0 0 0" rpy="${-M_PI/2} 0 ${-M_PI/2}" />
     <parent link="camera_rgb_frame" />
     <child link="camera_rgb_optical_frame" />

File: mobilebot_description/urdf/mobilebot.xacro (robot description, xacro)
@@ -261,59 +261,5 @@
 	</gazebo>
 <!-- kinect camera -->
-	<!-- <xacro:kinect xyz="0.150 0 0.037" parent_frame="top_plate" /> -->
-	<link name="camera_link">
-		<visual>
-			<origin xyz="0 0 0" rpy="0 0 1.570796"/>
-			<geometry>
-				<mesh filename="package://mobilebot_description/meshes/kinect.dae"/>
-			</geometry>
-		</visual>
-		<collision>
-			<origin xyz="0.0 0.0 0.0" rpy="0 0 0"/>
-			<geometry>
-				<box size="0.07271 0.27794 0.073"/>
-			</geometry>
-		</collision>
-		<inertial>
-			<mass value="0.564" />
-			<origin xyz="0 0 0" rpy="0 0 0"/>
-			<inertia ixx="0.003881243" ixy="0.0" ixz="0.0"
-								iyy="0.000498940" iyz="0.0"
-								izz="0.003879257" />
-		</inertial>
-  	</link>
-	<joint name="camera_joint" type="fixed">
-		<axis xyz="0 1 0" />
-		<origin xyz="0.150 0 0.037" rpy="0 0 0"/>
-		<parent link="top_plate"/>
-		<child link="camera_link"/>
-	</joint>
-	<joint name="camera_rgb_joint" type="fixed">
-		<!-- <origin xyz="-0.087 -0.0125 0.2870" rpy="0 0 0"/> -->
-		<origin xyz="-0.087 -0.0125 0.2870" rpy="0 0 0"/>
-		<parent link="camera_link"/>
-		<child link="camera_rgb_frame"/>
-	</joint>
-	<link name="camera_rgb_frame"/>
-	<joint name="camera_rgb_optical_joint" type="fixed">
-		<!-- <origin xyz="0 0 0" rpy="-1.570796 0 -1.570796" /> -->
-		<origin xyz="0 0 0" rpy="-1.570796 0 -1.570796" />
-		<parent link="camera_rgb_frame" />
-		<child link="camera_rgb_optical_frame" />
-	</joint>
-	<link name="camera_rgb_optical_frame"/>
-	<joint name="camera_depth_joint" type="fixed">
-		<origin xyz="0 -0.0250 0" rpy="0 0 0" />
-		<parent link="camera_rgb_frame" />
-		<child link="camera_depth_frame" />
-	</joint>
-	<link name="camera_depth_frame"/>
-	<joint name="camera_depth_optical_joint" type="fixed">
-		<!-- <origin xyz="0 0 0" rpy="-1.570796 0 -1.570796" /> -->
-		<origin xyz="0 0 0" rpy="-1.570796 0 -1.570796" />
-		<parent link="camera_depth_frame" />
-		<child link="camera_depth_optical_frame" />
-	</joint>
-	<link name="camera_depth_optical_frame" />
+	<xacro:kinect xyz="0.150 0 0.037" rpy="0 0 0" parent_frame="top_plate" />
 	<gazebo reference="camera_link">
 		<sensor type="depth" name="openni_camera">
